File: CCA0pre1.kicad_sch (KiCad schematic)
At the start: 0 parts

Commit message: Power Supply as in DSFigure 77
Parts:
- added C1: 10µF, symbol Device:C_Small
- added C10, C4, C6, C7, C8: 1µF, symbol Device:C_Small
- added C11: 100µF, symbol Device:C_Small
- added C2, C3, C5, C9: 0.1µF, symbol Device:C_Small
- added U1: ADS1299, Package_QFP:TQFP-64_10x10mm_P0.5mm, symbol Analog_ADC:ADS1299
Connections:
- new net: C8.1, C9.1, U1.55 (VCAP3)
- new net: C11.1, U1.28 (VCAP1)
- new net: C7.1, U1.26 (VCAP4)
- new net: C10.1, U1.30 (VCAP2)
- new net: C1.1, C2.1, U1.24 (VREFP)
- new net +3.3V: C5.1, C6.1, U1.48 (DVDD), U1.50 (DVDD)
- new net +5V: C3.2, C4.2, U1.19 (AVDD), U1.21 (AVDD), U1.22 (AVDD), U1.54 (AVDD1), U1.56 (AVDD), U1.59 (AVDD)
- new net GND: C1.2, C10.2, C11.2, C2.2, C3.1, C4.1, C5.2, C6.2, C7.2, C8.2, C9.2, U1.20 (AVSS), U1.23 (AVSS), U1.25 (VREFN), U1.31 (RESV1), U1.32 (AVSS), U1.33 (DGND), U1.49 (DGND), U1.51 (DGND), U1.53 (AVSS1), U1.57 (AVSS), U1.58 (AVSS)
Other:
- company: (none) -> MOVE- Prosthetics
- title: (none) -> ADS1299 pre 1
